File: pcb/ir-smart-led-controller.kicad_sch (KiCad schematic)
At the start: 7 parts, among them J1 Conn_01x03, U1 STM32G030J6Mx, U2 TSSP58038, U3 LDK220

Commit message: 0.0.1
Parts:
- C1, C2: value C -> 1uF
- C3: value C -> 100nF
Changed lines of the file:
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@@
       (effects (font (size 1.27 1.27)) (justify left))
     )
-    (property "Value" "C" (id 1) (at 86.995 99.6949 0)
+    (property "Value" "1uF" (id 1) (at 86.995 99.6949 0)
       (effects (font (size 1.27 1.27)) (justify left))
     )
@@
   (symbol (lib_id "Device:C") (at 113.665 97.79 0) (unit 1)
     (in_bom yes) (on_board yes) (fields_autoplaced)
-    (property "Reference" "C2" (id 0) (at 117.475 97.1549 0)
+    (property "Reference" "C2" (id 0) (at 116.84 97.1549 0)
       (effects (font (size 1.27 1.27)) (justify left))
     )
-    (property "Value" "C" (id 1) (at 117.475 99.6949 0)
+    (property "Value" "1uF" (id 1) (at 116.84 99.6949 0)
       (effects (font (size 1.27 1.27)) (justify left))
     )
@@
   (symbol (lib_id "Device:C") (at 122.555 97.79 0) (unit 1)
     (in_bom yes) (on_board yes) (fields_autoplaced)
-    (property "Reference" "C3" (id 0) (at 126.365 97.1549 0)
+    (property "Reference" "C3" (id 0) (at 125.73 97.1549 0)
       (effects (font (size 1.27 1.27)) (justify left))
     )
-    (property "Value" "C" (id 1) (at 126.365 99.6949 0)
+    (property "Value" "100nF" (id 1) (at 125.73 99.6949 0)
       (effects (font (size 1.27 1.27)) (justify left))
     )
@@
     )
     (path "/1bf4bfe3-f758-4a85-86f5-c84a6bd4f9e4"
-      (reference "C1") (unit 1) (value "C") (footprint "Capacitor_SMD:C_0603_1608Metric")
+      (reference "C1") (unit 1) (value "1uF") (footprint "Capacitor_SMD:C_0603_1608Metric")
     )
     (path "/62bfe1e6-8ccd-47e5-b825-7c8283629a85"
-      (reference "C2") (unit 1) (value "C") (footprint "Capacitor_SMD:C_0603_1608Metric")
+      (reference "C2") (unit 1) (value "1uF") (footprint "Capacitor_SMD:C_0603_1608Metric")
     )
     (path "/177f5fef-e824-4779-8085-3ad999ff3426"
-      (reference "C3") (unit 1) (value "C") (footprint "Capacitor_SMD:C_0603_1608Metric")
+      (reference "C3") (unit 1) (value "100nF") (footprint "Capacitor_SMD:C_0603_1608Metric")
     )
     (path "/f8374557-a6b3-432e-8e1f-c54fb7439493"

Commit message: update hal
Parts:
- ?: renamed from C3; value 100nF -> (none); footprint Capacitor_SMD:C_0603_1608Metric -> (none)
- ?: renamed from C1; value 1uF -> (none); footprint Capacitor_SMD:C_0603_1608Metric -> (none)
- ?: renamed from C2; value 1uF -> (none); footprint Capacitor_SMD:C_0603_1608Metric -> (none)
- ?: renamed from U1; value STM32G030J6Mx -> (none); footprint Package_SO:SOIC-8_3.9x4.9mm_P1.27mm -> (none)
- ?: renamed from U2; value TSSP58038 -> (none); footprint Connector_PinHeader_2.54mm:PinHeader_1x03_P2.54mm_Vertical -> (none)
- ?: renamed from J1; value Conn_01x03 -> (none); footprint Connector_PinHeader_2.54mm:PinHeader_1x03_P2.54mm_Vertical -> (none)
- ?: renamed from U3; value LDK220 -> (none); footprint Package_TO_SOT_SMD:SOT-23-5 -> (none)
